Commit message: Add configurable full syringe pump model and explicit TCP calibration gate

File: src/ur5e_toolheads/urdf/probe_tool.xacro (robot description, xacro)
@@ -7,4 +7,28 @@
   -->
   <xacro:macro name="probe_tool" params="parent_link">
+    <xacro:property name="pump" value="${xacro.load_yaml('$(find ur5e_toolheads)/config/printing_tool.yaml')}"/>
+    <xacro:if value="${pump['enabled']}">
+      <link name="probe_tool_link">
+        <visual>
+          <origin xyz="${'%s %s %s' % (pump['mesh_xyz'][0], pump['mesh_xyz'][1], pump['mesh_xyz'][2])}" rpy="${'%s %s %s' % (pump['mesh_rpy'][0], pump['mesh_rpy'][1], pump['mesh_rpy'][2])}"/>
+          <geometry><mesh filename="package://ur5e_toolheads/meshes/Full_UR_Syringe_Pump.stl" scale="${'%s %s %s' % (pump['mesh_scale'][0], pump['mesh_scale'][1], pump['mesh_scale'][2])}"/></geometry>
+          <material name="pump_gray"><color rgba="0.55 0.6 0.65 1"/></material>
+        </visual>
+        <collision>
+          <origin xyz="${'%s %s %s' % (pump['mesh_xyz'][0], pump['mesh_xyz'][1], pump['mesh_xyz'][2])}" rpy="${'%s %s %s' % (pump['mesh_rpy'][0], pump['mesh_rpy'][1], pump['mesh_rpy'][2])}"/>
+          <geometry><mesh filename="package://ur5e_toolheads/meshes/Full_UR_Syringe_Pump.stl" scale="${'%s %s %s' % (pump['mesh_scale'][0], pump['mesh_scale'][1], pump['mesh_scale'][2])}"/></geometry>
+        </collision>
+      </link>
+      <joint name="flange_to_probe_tool" type="fixed">
+        <parent link="${parent_link}"/><child link="probe_tool_link"/>
+        <origin xyz="${'%s %s %s' % (pump['mount_xyz'][0], pump['mount_xyz'][1], pump['mount_xyz'][2])}" rpy="${'%s %s %s' % (pump['mount_rpy'][0], pump['mount_rpy'][1], pump['mount_rpy'][2])}"/>
+      </joint>
+      <link name="probe_tcp"/>
+      <joint name="probe_tool_to_tcp" type="fixed">
+        <parent link="probe_tool_link"/><child link="probe_tcp"/>
+        <origin xyz="${'%s %s %s' % (pump['tcp_xyz'][0], pump['tcp_xyz'][1], pump['tcp_xyz'][2])}" rpy="${'%s %s %s' % (pump['tcp_rpy'][0], pump['tcp_rpy'][1], pump['tcp_rpy'][2])}"/>
+      </joint>
+    </xacro:if>
+    <xacro:unless value="${pump['enabled']}">
     <link name="probe_tool_link">
       <visual>
@@ -42,4 +66,9 @@
       <origin xyz="0 0 0.050032" rpy="0 0 0"/>
     </joint>
+    </xacro:unless>
+    <link name="nozzle_tcp"/>
+    <joint name="probe_tcp_to_nozzle_tcp" type="fixed">
+      <parent link="probe_tcp"/><child link="nozzle_tcp"/>
+    </joint>
   </xacro:macro>
 </robot>

Commit message: Add opt-in coarse pump collision envelopes for simulation demos

File: src/ur5e_toolheads/urdf/probe_tool.xacro (robot description, xacro)
@@ -15,9 +15,34 @@
           <material name="pump_gray"><color rgba="0.55 0.6 0.65 1"/></material>
         </visual>
+        <xacro:unless value="${pump.get('coarse_collision', False)}">
         <collision>
           <origin xyz="${'%s %s %s' % (pump['mesh_xyz'][0], pump['mesh_xyz'][1], pump['mesh_xyz'][2])}" rpy="${'%s %s %s' % (pump['mesh_rpy'][0], pump['mesh_rpy'][1], pump['mesh_rpy'][2])}"/>
           <geometry><mesh filename="package://ur5e_toolheads/meshes/Full_UR_Syringe_Pump.stl" scale="${'%s %s %s' % (pump['mesh_scale'][0], pump['mesh_scale'][1], pump['mesh_scale'][2])}"/></geometry>
         </collision>
+        </xacro:unless>
       </link>
+      <!-- Conservative envelopes in original CAD coordinates. Visual and TCP unchanged. -->
+      <xacro:if value="${pump.get('coarse_collision', False)}">
+        <link name="pump_sleeve_envelope">
+          <collision>
+            <origin xyz="0 ${1079.4*pump['mesh_scale'][1]} ${205.4*pump['mesh_scale'][2]}"/>
+            <geometry><cylinder radius="${53.0*max(pump['mesh_scale'][0],pump['mesh_scale'][1])}" length="${62.0*pump['mesh_scale'][2]}"/></geometry>
+          </collision>
+        </link>
+        <link name="pump_body_envelope">
+          <collision>
+            <origin xyz="${84.12483*pump['mesh_scale'][0]} ${1081.41265*pump['mesh_scale'][1]} ${199.14168*pump['mesh_scale'][2]}"/>
+            <geometry><box size="${83.25*pump['mesh_scale'][0]} ${43.0251*pump['mesh_scale'][1]} ${254.48336*pump['mesh_scale'][2]}"/></geometry>
+          </collision>
+        </link>
+        <joint name="tool_to_sleeve_envelope" type="fixed">
+          <parent link="probe_tool_link"/><child link="pump_sleeve_envelope"/>
+          <origin xyz="${'%s %s %s' % tuple(pump['mesh_xyz'])}" rpy="${'%s %s %s' % tuple(pump['mesh_rpy'])}"/>
+        </joint>
+        <joint name="tool_to_body_envelope" type="fixed">
+          <parent link="probe_tool_link"/><child link="pump_body_envelope"/>
+          <origin xyz="${'%s %s %s' % tuple(pump['mesh_xyz'])}" rpy="${'%s %s %s' % tuple(pump['mesh_rpy'])}"/>
+        </joint>
+      </xacro:if>
       <joint name="flange_to_probe_tool" type="fixed">
         <parent link="${parent_link}"/><child link="probe_tool_link"/>

Commit message: Fix coarse collision Xacro expressions without tuple builtin

File: src/ur5e_toolheads/urdf/probe_tool.xacro (robot description, xacro)
@@ -38,9 +38,9 @@
         <joint name="tool_to_sleeve_envelope" type="fixed">
           <parent link="probe_tool_link"/><child link="pump_sleeve_envelope"/>
-          <origin xyz="${'%s %s %s' % tuple(pump['mesh_xyz'])}" rpy="${'%s %s %s' % tuple(pump['mesh_rpy'])}"/>
+          <origin xyz="${'%s %s %s' % (pump['mesh_xyz'][0], pump['mesh_xyz'][1], pump['mesh_xyz'][2])}" rpy="${'%s %s %s' % (pump['mesh_rpy'][0], pump['mesh_rpy'][1], pump['mesh_rpy'][2])}"/>
         </joint>
         <joint name="tool_to_body_envelope" type="fixed">
           <parent link="probe_tool_link"/><child link="pump_body_envelope"/>
-          <origin xyz="${'%s %s %s' % tuple(pump['mesh_xyz'])}" rpy="${'%s %s %s' % tuple(pump['mesh_rpy'])}"/>
+          <origin xyz="${'%s %s %s' % (pump['mesh_xyz'][0], pump['mesh_xyz'][1], pump['mesh_xyz'][2])}" rpy="${'%s %s %s' % (pump['mesh_rpy'][0], pump['mesh_rpy'][1], pump['mesh_rpy'][2])}"/>
         </joint>
       </xacro:if>

Commit message: Tighten coarse pump envelope near surface-facing outlet

File: src/ur5e_toolheads/urdf/probe_tool.xacro (robot description, xacro)
@@ -32,6 +32,32 @@
         <link name="pump_body_envelope">
           <collision>
-            <origin xyz="${84.12483*pump['mesh_scale'][0]} ${1081.41265*pump['mesh_scale'][1]} ${199.14168*pump['mesh_scale'][2]}"/>
-            <geometry><box size="${83.25*pump['mesh_scale'][0]} ${43.0251*pump['mesh_scale'][1]} ${254.48336*pump['mesh_scale'][2]}"/></geometry>
+            <!-- Main body stops before the narrow dispensing end. -->
+            <origin xyz="${84.12483*pump['mesh_scale'][0]} ${1081.41265*pump['mesh_scale'][1]} ${173.7*pump['mesh_scale'][2]}"/>
+            <geometry><box size="${83.25*pump['mesh_scale'][0]} ${43.0251*pump['mesh_scale'][1]} ${203.6*pump['mesh_scale'][2]}"/></geometry>
+          </collision>
+        </link>
+        <!-- Tighter primitives follow the STL near the TCP. -->
+        <link name="pump_tip_stem_envelope">
+          <collision>
+            <origin xyz="${87.65*pump['mesh_scale'][0]} ${1083.25*pump['mesh_scale'][1]} ${293.6*pump['mesh_scale'][2]}"/>
+            <geometry><box size="${3.9*pump['mesh_scale'][0]} ${12.3*pump['mesh_scale'][1]} ${34.6*pump['mesh_scale'][2]}"/></geometry>
+          </collision>
+        </link>
+        <link name="pump_tip_collar_envelope">
+          <collision>
+            <origin xyz="${96.74983*pump['mesh_scale'][0]} ${1081.4002*pump['mesh_scale'][1]} ${313.05*pump['mesh_scale'][2]}"/>
+            <geometry><cylinder radius="${11.0*max(pump['mesh_scale'][0],pump['mesh_scale'][1])}" length="${4.5*pump['mesh_scale'][2]}"/></geometry>
+          </collision>
+        </link>
+        <link name="pump_nozzle_envelope">
+          <collision>
+            <origin xyz="${96.74983*pump['mesh_scale'][0]} ${1081.4002*pump['mesh_scale'][1]} ${319.25*pump['mesh_scale'][2]}"/>
+            <geometry><cylinder radius="${5.0*max(pump['mesh_scale'][0],pump['mesh_scale'][1])}" length="${8.5*pump['mesh_scale'][2]}"/></geometry>
+          </collision>
+        </link>
+        <link name="pump_outlet_envelope">
+          <collision>
+            <origin xyz="${96.74983*pump['mesh_scale'][0]} ${1081.4002*pump['mesh_scale'][1]} ${324.55*pump['mesh_scale'][2]}"/>
+            <geometry><cylinder radius="${2.2*max(pump['mesh_scale'][0],pump['mesh_scale'][1])}" length="${3.0*pump['mesh_scale'][2]}"/></geometry>
           </collision>
         </link>
@@ -42,4 +68,20 @@
         <joint name="tool_to_body_envelope" type="fixed">
           <parent link="probe_tool_link"/><child link="pump_body_envelope"/>
+          <origin xyz="${'%s %s %s' % (pump['mesh_xyz'][0], pump['mesh_xyz'][1], pump['mesh_xyz'][2])}" rpy="${'%s %s %s' % (pump['mesh_rpy'][0], pump['mesh_rpy'][1], pump['mesh_rpy'][2])}"/>
+        </joint>
+        <joint name="tool_to_tip_stem_envelope" type="fixed">
+          <parent link="probe_tool_link"/><child link="pump_tip_stem_envelope"/>
+          <origin xyz="${'%s %s %s' % (pump['mesh_xyz'][0], pump['mesh_xyz'][1], pump['mesh_xyz'][2])}" rpy="${'%s %s %s' % (pump['mesh_rpy'][0], pump['mesh_rpy'][1], pump['mesh_rpy'][2])}"/>
+        </joint>
+        <joint name="tool_to_tip_collar_envelope" type="fixed">
+          <parent link="probe_tool_link"/><child link="pump_tip_collar_envelope"/>
+          <origin xyz="${'%s %s %s' % (pump['mesh_xyz'][0], pump['mesh_xyz'][1], pump['mesh_xyz'][2])}" rpy="${'%s %s %s' % (pump['mesh_rpy'][0], pump['mesh_rpy'][1], pump['mesh_rpy'][2])}"/>
+        </joint>
+        <joint name="tool_to_nozzle_envelope" type="fixed">
+          <parent link="probe_tool_link"/><child link="pump_nozzle_envelope"/>
+          <origin xyz="${'%s %s %s' % (pump['mesh_xyz'][0], pump['mesh_xyz'][1], pump['mesh_xyz'][2])}" rpy="${'%s %s %s' % (pump['mesh_rpy'][0], pump['mesh_rpy'][1], pump['mesh_rpy'][2])}"/>
+        </joint>
+        <joint name="tool_to_outlet_envelope" type="fixed">
+          <parent link="probe_tool_link"/><child link="pump_outlet_envelope"/>
           <origin xyz="${'%s %s %s' % (pump['mesh_xyz'][0], pump['mesh_xyz'][1], pump['mesh_xyz'][2])}" rpy="${'%s %s %s' % (pump['mesh_rpy'][0], pump['mesh_rpy'][1], pump['mesh_rpy'][2])}"/>
         </joint>

Commit message: Separate coarse pump body from wrist sleeve

File: src/ur5e_toolheads/urdf/probe_tool.xacro (robot description, xacro)
@@ -32,7 +32,12 @@
         <link name="pump_body_envelope">
           <collision>
-            <!-- Main body stops before the narrow dispensing end. -->
-            <origin xyz="${84.12483*pump['mesh_scale'][0]} ${1081.41265*pump['mesh_scale'][1]} ${173.7*pump['mesh_scale'][2]}"/>
-            <geometry><box size="${83.25*pump['mesh_scale'][0]} ${43.0251*pump['mesh_scale'][1]} ${203.6*pump['mesh_scale'][2]}"/></geometry>
+            <!--
+              The sleeve owns the flange-adjacent region out to CAD X=53 mm.
+              Start the checked body at that boundary so its conservative box
+              cannot permanently overlap wrist_2 through the sleeve.  The far
+              face remains at the STL bound X=125.25 mm.
+            -->
+            <origin xyz="${89.125*pump['mesh_scale'][0]} ${1081.41265*pump['mesh_scale'][1]} ${173.7*pump['mesh_scale'][2]}"/>
+            <geometry><box size="${72.25*pump['mesh_scale'][0]} ${43.0251*pump['mesh_scale'][1]} ${203.6*pump['mesh_scale'][2]}"/></geometry>
           </collision>
         </link>

Commit message: Add clearance at coarse wrist sleeve boundary

File: src/ur5e_toolheads/urdf/probe_tool.xacro (robot description, xacro)
@@ -27,5 +27,5 @@
           <collision>
             <origin xyz="0 ${1079.4*pump['mesh_scale'][1]} ${205.4*pump['mesh_scale'][2]}"/>
-            <geometry><cylinder radius="${53.0*max(pump['mesh_scale'][0],pump['mesh_scale'][1])}" length="${62.0*pump['mesh_scale'][2]}"/></geometry>
+            <geometry><cylinder radius="${54.0*max(pump['mesh_scale'][0],pump['mesh_scale'][1])}" length="${62.0*pump['mesh_scale'][2]}"/></geometry>
           </collision>
         </link>
@@ -33,11 +33,11 @@
           <collision>
             <!--
-              The sleeve owns the flange-adjacent region out to CAD X=53 mm.
+              The sleeve owns the flange-adjacent region out to CAD X=54 mm.
               Start the checked body at that boundary so its conservative box
               cannot permanently overlap wrist_2 through the sleeve.  The far
               face remains at the STL bound X=125.25 mm.
             -->
-            <origin xyz="${89.125*pump['mesh_scale'][0]} ${1081.41265*pump['mesh_scale'][1]} ${173.7*pump['mesh_scale'][2]}"/>
-            <geometry><box size="${72.25*pump['mesh_scale'][0]} ${43.0251*pump['mesh_scale'][1]} ${203.6*pump['mesh_scale'][2]}"/></geometry>
+            <origin xyz="${89.625*pump['mesh_scale'][0]} ${1081.41265*pump['mesh_scale'][1]} ${173.7*pump['mesh_scale'][2]}"/>
+            <geometry><box size="${71.25*pump['mesh_scale'][0]} ${43.0251*pump['mesh_scale'][1]} ${203.6*pump['mesh_scale'][2]}"/></geometry>
           </collision>
         </link>

Commit message: Model thin needle extension in tool collisions

File: src/ur5e_toolheads/urdf/probe_tool.xacro (robot description, xacro)
@@ -67,4 +67,17 @@
           </collision>
         </link>
+        <xacro:if value="${pump.get('needle_length_mm', 0.0) > 0.0}">
+          <link name="pump_needle_envelope">
+            <visual>
+              <origin xyz="${pump['syringe_outlet_cad_mm'][0]*pump['mesh_scale'][0]} ${pump['syringe_outlet_cad_mm'][1]*pump['mesh_scale'][1]} ${pump['syringe_outlet_cad_mm'][2]*pump['mesh_scale'][2]+(pump['needle_length_mm']-pump.get('needle_collision_tip_clearance_mm',2.0))/2000.0}"/>
+              <geometry><cylinder radius="${pump.get('needle_radius_mm',1.0)/1000.0}" length="${(pump['needle_length_mm']-pump.get('needle_collision_tip_clearance_mm',2.0))/1000.0}"/></geometry>
+              <material name="needle_metal"><color rgba="0.72 0.75 0.78 1"/></material>
+            </visual>
+            <collision>
+              <origin xyz="${pump['syringe_outlet_cad_mm'][0]*pump['mesh_scale'][0]} ${pump['syringe_outlet_cad_mm'][1]*pump['mesh_scale'][1]} ${pump['syringe_outlet_cad_mm'][2]*pump['mesh_scale'][2]+(pump['needle_length_mm']-pump.get('needle_collision_tip_clearance_mm',2.0))/2000.0}"/>
+              <geometry><cylinder radius="${pump.get('needle_radius_mm',1.0)/1000.0}" length="${(pump['needle_length_mm']-pump.get('needle_collision_tip_clearance_mm',2.0))/1000.0}"/></geometry>
+            </collision>
+          </link>
+        </xacro:if>
         <joint name="tool_to_sleeve_envelope" type="fixed">
           <parent link="probe_tool_link"/><child link="pump_sleeve_envelope"/>
@@ -91,4 +104,10 @@
           <origin xyz="${'%s %s %s' % (pump['mesh_xyz'][0], pump['mesh_xyz'][1], pump['mesh_xyz'][2])}" rpy="${'%s %s %s' % (pump['mesh_rpy'][0], pump['mesh_rpy'][1], pump['mesh_rpy'][2])}"/>
         </joint>
+        <xacro:if value="${pump.get('needle_length_mm', 0.0) > 0.0}">
+          <joint name="tool_to_needle_envelope" type="fixed">
+            <parent link="probe_tool_link"/><child link="pump_needle_envelope"/>
+            <origin xyz="${'%s %s %s' % (pump['mesh_xyz'][0], pump['mesh_xyz'][1], pump['mesh_xyz'][2])}" rpy="${'%s %s %s' % (pump['mesh_rpy'][0], pump['mesh_rpy'][1], pump['mesh_rpy'][2])}"/>
+          </joint>
+        </xacro:if>
       </xacro:if>
       <joint name="flange_to_probe_tool" type="fixed">

Commit message: Separate needle and outlet collision envelopes

File: src/ur5e_toolheads/urdf/probe_tool.xacro (robot description, xacro)
@@ -70,11 +70,11 @@
           <link name="pump_needle_envelope">
             <visual>
-              <origin xyz="${pump['syringe_outlet_cad_mm'][0]*pump['mesh_scale'][0]} ${pump['syringe_outlet_cad_mm'][1]*pump['mesh_scale'][1]} ${pump['syringe_outlet_cad_mm'][2]*pump['mesh_scale'][2]+(pump['needle_length_mm']-pump.get('needle_collision_tip_clearance_mm',2.0))/2000.0}"/>
-              <geometry><cylinder radius="${pump.get('needle_radius_mm',1.0)/1000.0}" length="${(pump['needle_length_mm']-pump.get('needle_collision_tip_clearance_mm',2.0))/1000.0}"/></geometry>
+              <origin xyz="${pump['syringe_outlet_cad_mm'][0]*pump['mesh_scale'][0]} ${pump['syringe_outlet_cad_mm'][1]*pump['mesh_scale'][1]} ${pump['syringe_outlet_cad_mm'][2]*pump['mesh_scale'][2]+(pump.get('needle_collision_base_clearance_mm',1.0)+(pump['needle_length_mm']-pump.get('needle_collision_base_clearance_mm',1.0)-pump.get('needle_collision_tip_clearance_mm',2.0))/2.0)/1000.0}"/>
+              <geometry><cylinder radius="${pump.get('needle_radius_mm',1.0)/1000.0}" length="${(pump['needle_length_mm']-pump.get('needle_collision_base_clearance_mm',1.0)-pump.get('needle_collision_tip_clearance_mm',2.0))/1000.0}"/></geometry>
               <material name="needle_metal"><color rgba="0.72 0.75 0.78 1"/></material>
             </visual>
             <collision>
-              <origin xyz="${pump['syringe_outlet_cad_mm'][0]*pump['mesh_scale'][0]} ${pump['syringe_outlet_cad_mm'][1]*pump['mesh_scale'][1]} ${pump['syringe_outlet_cad_mm'][2]*pump['mesh_scale'][2]+(pump['needle_length_mm']-pump.get('needle_collision_tip_clearance_mm',2.0))/2000.0}"/>
-              <geometry><cylinder radius="${pump.get('needle_radius_mm',1.0)/1000.0}" length="${(pump['needle_length_mm']-pump.get('needle_collision_tip_clearance_mm',2.0))/1000.0}"/></geometry>
+              <origin xyz="${pump['syringe_outlet_cad_mm'][0]*pump['mesh_scale'][0]} ${pump['syringe_outlet_cad_mm'][1]*pump['mesh_scale'][1]} ${pump['syringe_outlet_cad_mm'][2]*pump['mesh_scale'][2]+(pump.get('needle_collision_base_clearance_mm',1.0)+(pump['needle_length_mm']-pump.get('needle_collision_base_clearance_mm',1.0)-pump.get('needle_collision_tip_clearance_mm',2.0))/2.0)/1000.0}"/>
+              <geometry><cylinder radius="${pump.get('needle_radius_mm',1.0)/1000.0}" length="${(pump['needle_length_mm']-pump.get('needle_collision_base_clearance_mm',1.0)-pump.get('needle_collision_tip_clearance_mm',2.0))/1000.0}"/></geometry>
             </collision>
           </link>

Commit message: Add manually positioned tube printing and axial 160 mm nozzle TCP
Capture fresh live nozzle state, generate a fixed-orientation nominal 10 mm helix, and reuse guarded saved-plan execution. Preserve pump collision geometry and require physical calibration verification. Add TCP composition and tube geometry tests plus host setup commands.

File: src/ur5e_toolheads/urdf/probe_tool.xacro (robot description, xacro)
@@ -8,4 +8,22 @@
   <xacro:macro name="probe_tool" params="parent_link">
     <xacro:property name="pump" value="${xacro.load_yaml('$(find ur5e_toolheads)/config/printing_tool.yaml')}"/>
+    <!-- Total flange-to-tip nozzle, independent of the old CAD outlet offset. -->
+    <xacro:if value="${pump['enabled'] and pump.get('axial_nozzle_length_mm',0.0) > 0.0}">
+      <link name="axial_nozzle_envelope">
+        <visual>
+          <origin xyz="${pump['axial_nozzle_length_mm']/2000.0} 0 0" rpy="${pi/2} 0 ${pi/2}"/>
+          <geometry><cylinder radius="${pump['axial_nozzle_radius_mm']/1000.0}" length="${pump['axial_nozzle_length_mm']/1000.0}"/></geometry>
+          <material name="axial_nozzle_metal"><color rgba="0.72 0.75 0.78 1"/></material>
+        </visual>
+        <collision>
+          <!-- Last 0.5 mm is the intended deposition/contact zone. -->
+          <origin xyz="${(pump['axial_nozzle_length_mm']-0.5)/2000.0} 0 0" rpy="${pi/2} 0 ${pi/2}"/>
+          <geometry><cylinder radius="${pump['axial_nozzle_radius_mm']/1000.0}" length="${(pump['axial_nozzle_length_mm']-0.5)/1000.0}"/></geometry>
+        </collision>
+      </link>
+      <joint name="flange_to_axial_nozzle" type="fixed">
+        <parent link="${parent_link}"/><child link="axial_nozzle_envelope"/>
+      </joint>
+    </xacro:if>
     <xacro:if value="${pump['enabled']}">
       <link name="probe_tool_link">
